File: Schematics/control_board.brd (EAGLE design)
At the start: 160 x 100 mm, 1 part

Commit message: Added some of the dimmer switch circuit
Parts:
- added R1, R2: 15K, ref_lib:YAG5755-ND
- added R3: 1.5K, ref_lib:CR-25
- added R4: 220, ref_lib:CR-25
- added U$1: QG015L5TP, ref_lib:QG015L5TP
- added U1: H11AA4M, thermo:H11AA4M
- added U2: MOC3052M, thermo:MOC3052M
- moved A1 26.2 mm to (26.7, 14.0)
Connections:
- new net GND: U1.E, U2.IN2
- new net N$1: R1.P$1, U1.IN2
- new net N$2: R2.P$1, U1.IN1
- new net N$3: R2.P$2, U$1.P$3
- new net N$4: R1.P$2
- new net N$5: R3.P$1, U2.MAIN@2
- new net N$6: R3.P$2, U$1.P$2
- new net N$7: R4.P$2, U2.IN1
Changed lines of the file:
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@@
 </autorouter>
 <elements>
-<element name="A1" library="Arduino" package="NANO_EVERY_SOCKET" value="NANO_EVERY" x="20.32" y="-11.43" smashed="yes">
-<attribute name="NAME" x="13.97" y="-12.7" size="2.54" layer="21"/>
+<element name="A1" library="Arduino" package="NANO_EVERY_SOCKET" value="NANO_EVERY" x="26.67" y="13.97" smashed="yes">
+<attribute name="NAME" x="20.32" y="12.7" size="2.54" layer="21"/>
+</element>
+<element name="U1" library="thermo" package="H11AA4M" value="H11AA4M" x="91.44" y="8.89" smashed="yes">
+<attribute name="NAME" x="88.07" y="7.07" size="1.27" layer="21"/>
+</element>
+<element name="U2" library="thermo" package="MOC3052M" value="MOC3052M" x="71.12" y="10.16" smashed="yes">
+<attribute name="NAME" x="67.75" y="8.34" size="1.27" layer="21"/>
+</element>
+<element name="R1" library="ref_lib" package="YAG5755-ND" value="15K" x="67.31" y="44.45" smashed="yes">
+<attribute name="NAME" x="64.31" y="48.45" size="1.27" layer="21"/>
+<attribute name="VALUE" x="64.31" y="39.45" size="1.27" layer="21"/>
+</element>
+<element name="R2" library="ref_lib" package="YAG5755-ND" value="15K" x="90.17" y="33.02" smashed="yes">
+<attribute name="NAME" x="87.17" y="37.02" size="1.27" layer="21"/>
+<attribute name="VALUE" x="87.17" y="28.02" size="1.27" layer="21"/>
+</element>
+<element name="U$1" library="ref_lib" package="QG015L5TP" value="QG015L5TP" x="-13.97" y="-22.86" smashed="yes"/>
+<element name="R3" library="ref_lib" package="CR-25" value="1.5K" x="17.78" y="41.91" smashed="yes">
+<attribute name="NAME" x="15.08" y="41.11" size="0.6096" layer="21"/>
+<attribute name="VALUE" x="15.08" y="42.11" size="0.6096" layer="21"/>
+</element>
+<element name="R4" library="ref_lib" package="CR-25" value="220" x="-25.4" y="-6.35" smashed="yes">
+<attribute name="NAME" x="-28.1" y="-7.15" size="0.6096" layer="21"/>
+<attribute name="VALUE" x="-28.1" y="-6.15" size="0.6096" layer="21"/>
 </element>
 </elements>
@@
 <contactref element="A1" pad="VIN"/>
 </signal>
+<signal name="GND">
+<contactref element="U2" pad="IN2"/>
+<contactref element="U1" pad="E"/>
+<wire x1="93.98" y1="12.7" x2="71.12" y2="6.35" width="0" layer="19" extent="1-1"/>
+</signal>
+<signal name="N$1">
+<contactref element="R1" pad="P$1"/>
+<contactref element="U1" pad="IN2"/>
+<wire x1="91.44" y1="5.08" x2="50.31" y2="44.45" width="0" layer="19" extent="1-1"/>
+</signal>
+<signal name="N$2">
+<contactref element="R2" pad="P$1"/>
+<contactref element="U1" pad="IN1"/>
+<wire x1="88.9" y1="5.08" x2="73.17" y2="33.02" width="0" layer="19" extent="1-1"/>
+</signal>
+<signal name="N$3">
+<contactref element="U$1" pad="P$3"/>
+<contactref element="R2" pad="P$2"/>
+<wire x1="107.17" y1="33.02" x2="-16.51" y2="-22.86" width="0" layer="19" extent="1-1"/>
+</signal>
+<signal name="N$4">
+<contactref element="R1" pad="P$2"/>
+</signal>
+<signal name="N$5">
+<contactref element="U2" pad="MAIN@2"/>
+<contactref element="R3" pad="P$1"/>
+<wire x1="73.66" y1="13.97" x2="11.78" y2="41.91" width="0" layer="19" extent="1-1"/>
+</signal>
+<signal name="N$6">
+<contactref element="R3" pad="P$2"/>
+<contactref element="U$1" pad="P$2"/>
+<wire x1="23.78" y1="41.91" x2="-13.97" y2="-22.86" width="0" layer="19" extent="1-1"/>
+</signal>
+<signal name="N$7">
+<contactref element="R4" pad="P$2"/>
+<contactref element="U2" pad="IN1"/>
+<wire x1="68.58" y1="6.35" x2="-19.4" y2="-6.35" width="0" layer="19" extent="1-1"/>
+</signal>
 </signals>

Commit message: Rev 1.0
Parts:
- removed A1: NANO_EVERY, Arduino:NANO_EVERY_SOCKET
- added CN1, CN2: MOLEX-BEAU-BARRIER-2, ref_lib:MOLEX-BEAU-BARRIER-2
- added JP1: (no value), pinhead:1X03/90
- R1, R2: device ref_lib:YAG5755-ND -> ref_lib:RSF100
- moved U1 77.6 mm to (14.0, 12.7), turned to 90 degrees
- moved U$1 65.7 mm to (35.6, 20.3)
- moved R2 46.0 mm to (48.3, 14.0)
- moved R1 42.6 mm to (48.3, 6.35), turned to 180 degrees
- moved U2 42.2 mm to (29.2, 5.08), turned to 270 degrees
- moved R4 41.0 mm to (14.0, 5.08)
- moved R3 28.5 mm to (27.9, 15.2)
Connections:
- removed net N$3: R2.P$2, U$1.P$3
- removed net N$4: R1.P$2
- removed net VIN: A1.VIN
- new net CONTROL: JP1.2, R4.P$1
- new net CROSSOVER: JP1.3, U1.C
- new net HEATER-OUT: CN2.P1, U$1.P$1
- new net LIVE: CN1.P1, R1.P$2, U$1.P$3, U2.MAIN@1
- new net NEUTRAL: CN1.P2, CN2.P2, R2.P$2
- net GND: now also JP1.1
- net N$1: now also R2.P$1; no longer R1.P$1
- net N$2: now also R1.P$1; no longer R2.P$1
Routing:
- net LIVE: track 0.00 -> 49.2 mm
- net N$2: track 0.00 -> 42.4 mm, vias 0 -> 2
- net GND: track 0.00 -> 31.8 mm
- net HEATER-OUT: track 0.00 -> 27.1 mm
- net N$1: track 0.00 -> 25.8 mm, vias 0 -> 2
- net N$5: track 0.00 -> 17.6 mm
- net CROSSOVER: track 0.00 -> 7.44 mm
- net N$7: track 0.00 -> 6.48 mm
- net N$6: track 0.00 -> 5.78 mm
- net CONTROL: track 0.00 -> 5.21 mm
- added copper zone on layer 16, net NEUTRAL
Other:
- board size 160 x 100 mm -> 60 x 52 mm
- board text added: "Heat-Pad Power Board"
- board text added: "Rev 1.0"

Commit message: I can definitely read spec sheets.
Connections:
- net HEATER-OUT: now also U$1.P$3; no longer U$1.P$1
- net LIVE: now also U$1.P$2; no longer U$1.P$3
- net N$6: now also U$1.P$1; no longer U$1.P$2
Routing:
- net N$1: track 25.8 -> 38.4 mm, vias 2 -> 0
- net LIVE: track 49.2 -> 56.4 mm, vias 0 -> 1
- net HEATER-OUT: track 27.1 -> 29.6 mm, vias 0 -> 1
- net N$6: track 5.78 -> 6.87 mm, vias 0 -> 1
- net N$2: track 42.4 -> 42.9 mm, vias 2 -> 1
Other:
- board text added: "Prototype Not Safety Rated"
