File: Schematics/control_board.sch (EAGLE design)
At the start: 1 part

Commit message: Added some of the dimmer switch circuit
Parts:
- added R1, R2: 15K, ref_lib:YAG5755-ND
- added R3: 1.5K, ref_lib:YAGEO_CFR
- added R4: 220, ref_lib:YAGEO_CFR
- added U$1: QG015L5TP, ref_lib:QG015L5TP
- added U1: H11AA4M, thermo:H11AA4M
- added U2: MOC3052M, thermo:MOC3052M
Connections:
- new net GND: U1.E, U2.IN2
- new net N$1: R1.1, U1.IN2
- new net N$2: R2.1, U1.IN1
- new net N$3: R2.2, U$1.A2
- new net N$4: R1.2
- new net N$5: R3.1, U2.MAIN@2
- new net N$6: R3.2, U$1.G
- new net N$7: R4.2, U2.IN1
Other:
- note added: "TODO: This should probably be a power resistor."
Changed lines of the file:
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@@
 <parts>
 <part name="A1" library="Arduino" deviceset="NANO_EVERY" device=""/>
+<part name="U1" library="thermo" deviceset="H11AA4M" device=""/>
+<part name="U2" library="thermo" deviceset="MOC3052M" device=""/>
+<part name="R1" library="ref_lib" deviceset="YAG5755-ND" device="" value="15K"/>
+<part name="R2" library="ref_lib" deviceset="YAG5755-ND" device="" value="15K"/>
+<part name="U$1" library="ref_lib" deviceset="QG015L5TP" device=""/>
+<part name="R3" library="ref_lib" deviceset="YAGEO_CFR" device="" value="1.5K"/>
+<part name="R4" library="ref_lib" deviceset="YAGEO_CFR" device="" value="220"/>
 </parts>
 <sheets>
@@
 </nets>
 </sheet>
+<sheet>
+<description>HighPower</description>
+<plain>
+<text x="83.82" y="25.4" size="1.778" layer="91">TODO: This should probably be a power resistor.</text>
+</plain>
+<instances>
+<instance part="U1" gate="G$1" x="55.88" y="76.2" smashed="yes">
+<attribute name="NAME" x="48.26" y="66.04" size="1.27" layer="94"/>
+</instance>
+<instance part="U2" gate="G$1" x="55.88" y="40.64" smashed="yes">
+<attribute name="NAME" x="48.26" y="30.48" size="1.27" layer="94"/>
+</instance>
+<instance part="R1" gate="G$1" x="78.74" y="99.06" smashed="yes">
+<attribute name="NAME" x="74.93" y="100.5586" size="1.778" layer="95"/>
+<attribute name="VALUE" x="74.93" y="95.758" size="1.778" layer="96"/>
+</instance>
+<instance part="R2" gate="G$1" x="78.74" y="91.44" smashed="yes">
+<attribute name="NAME" x="74.93" y="92.9386" size="1.778" layer="95"/>
+<attribute name="VALUE" x="74.93" y="88.138" size="1.778" layer="96"/>
+</instance>
+<instance part="U$1" gate="G$1" x="111.76" y="35.56" smashed="yes">
+<attribute name="NAME" x="115.57" y="38.1" size="1.778" layer="95"/>
+<attribute name="VALUE" x="115.57" y="35.56" size="1.778" layer="96"/>
+</instance>
+<instance part="R3" gate="G$1" x="88.9" y="35.56" smashed="yes">
+<attribute name="NAME" x="85.09" y="37.0586" size="1.778" layer="95"/>
+<attribute name="VALUE" x="85.09" y="32.258" size="1.778" layer="96"/>
+</instance>
+<instance part="R4" gate="G$1" x="15.24" y="45.72" smashed="yes">
+<attribute name="NAME" x="11.43" y="47.2186" size="1.778" layer="95"/>
+<attribute name="VALUE" x="11.43" y="42.418" size="1.778" layer="96"/>
+</instance>
+</instances>
+<busses>
+</busses>
+<nets>
+<net name="GND" class="0">
+<segment>
+<pinref part="U2" gate="G$1" pin="IN2"/>
+<wire x1="43.18" y1="40.64" x2="30.48" y2="40.64" width="0.1524" layer="91"/>
+<label x="30.48" y="40.64" size="1.778" layer="95"/>
+</segment>
+<segment>
+<pinref part="U1" gate="G$1" pin="E"/>
+<wire x1="68.58" y1="71.12" x2="81.28" y2="71.12" width="0.1524" layer="91"/>
+<label x="76.2" y="71.12" size="1.778" layer="95"/>
+</segment>
+</net>
+<net name="N$1" class="0">
+<segment>
+<pinref part="R1" gate="G$1" pin="1"/>
+<wire x1="73.66" y1="99.06" x2="30.48" y2="99.06" width="0.1524" layer="91"/>
+<wire x1="30.48" y1="99.06" x2="30.48" y2="76.2" width="0.1524" layer="91"/>
+<pinref part="U1" gate="G$1" pin="IN2"/>
+<wire x1="30.48" y1="76.2" x2="43.18" y2="76.2" width="0.1524" layer="91"/>
+</segment>
+</net>
+<net name="N$2" class="0">
+<segment>
+<pinref part="R2" gate="G$1" pin="1"/>
+<wire x1="73.66" y1="91.44" x2="38.1" y2="91.44" width="0.1524" layer="91"/>
+<wire x1="38.1" y1="91.44" x2="38.1" y2="81.28" width="0.1524" layer="91"/>
+<pinref part="U1" gate="G$1" pin="IN1"/>
+<wire x1="38.1" y1="81.28" x2="43.18" y2="81.28" width="0.1524" layer="91"/>
+</segment>
+</net>
+<net name="N$3" class="0">
+<segment>
+<pinref part="U$1" gate="G$1" pin="A2"/>
+<pinref part="R2" gate="G$1" pin="2"/>
+<wire x1="111.76" y1="40.64" x2="111.76" y2="45.72" width="0.1524" layer="91"/>
+<wire x1="111.76" y1="45.72" x2="111.76" y2="91.44" width="0.1524" layer="91"/>
+<wire x1="111.76" y1="91.44" x2="83.82" y2="91.44" width="0.1524" layer="91"/>
+<wire x1="71.12" y1="45.72" x2="111.76" y2="45.72" width="0.1524" layer="91"/>
+<junction x="111.76" y="45.72"/>
+</segment>
+</net>
+<net name="N$4" class="0">
+<segment>
+<pinref part="R1" gate="G$1" pin="2"/>
+<wire x1="83.82" y1="99.06" x2="111.76" y2="99.06" width="0.1524" layer="91"/>
+</segment>
+</net>
+<net name="N$5" class="0">
+<segment>
+<pinref part="U2" gate="G$1" pin="MAIN@2"/>
+<pinref part="R3" gate="G$1" pin="1"/>
+<wire x1="68.58" y1="35.56" x2="83.82" y2="35.56" width="0.1524" layer="91"/>
+</segment>
+</net>
+<net name="N$6" class="0">
+<segment>
+<pinref part="R3" gate="G$1" pin="2"/>
+<pinref part="U$1" gate="G$1" pin="G"/>
+<wire x1="93.98" y1="35.56" x2="106.68" y2="35.56" width="0.1524" layer="91"/>
+</segment>
+</net>
+<net name="N$7" class="0">
+<segment>
+<pinref part="R4" gate="G$1" pin="2"/>
+<pinref part="U2" gate="G$1" pin="IN1"/>
+<wire x1="20.32" y1="45.72" x2="43.18" y2="45.72" width="0.1524" layer="91"/>
+</segment>
+</net>
+</nets>
+</sheet>

Commit message: Rev 1.0
Parts:
- removed A1: NANO_EVERY, Arduino:NANO_EVERY
- added CN1, CN2: MOLEX-BEAU-BARRIER-2, ref_lib:MOLEX-BEAU-BARRIER-2
- added JP1: (no value), pinhead:PINHD-1X3/90
- R1, R2: device ref_lib:YAG5755-ND -> ref_lib:RSF100JB-73
Connections:
- removed net N$3: R2.2, U$1.A2
- removed net N$4: R1.2
- new net CONTROL: JP1.2, R4.1
- new net CROSSOVER: JP1.3, U1.C
- new net HEATER-OUT: CN2.1, U$1.A1
- new net LIVE: CN1.1, R1.2, U$1.A2, U2.MAIN@1
- new net NEUTRAL: CN1.2, CN2.2, R2.2
- net GND: now also JP1.1
- net N$1: now also R2.1; no longer R1.1
- net N$2: now also R1.1; no longer R2.1
